Commit message: added world files and adjusted launcher

File: description/wheelchair_backrest.xacro (robot description, xacro)
@@ -27,5 +27,5 @@
         <!-- FOR EVERY VISUAL, INCLUDE THE FOLLOWING TO REFLECT IT ON GAZEBO -->
         <gazebo reference="${name}">
-            <material value="Gazebo/White"/>
+            <material value="Gazebo/Grey"/>
         </gazebo>
     </xacro:macro>

File: description/wheelchair_castor_wheel.xacro (robot description, xacro)
@@ -33,5 +33,5 @@
         </link>
         <gazebo reference="${side}_castor_wheel">
-            <material value="Gazebo/Black"/>
+            <material value="Gazebo/Orange"/>
             <!-- Trick to make the caster wheel w/o (negligible) friction.. trick -->
             <mu1 value="0.001"/>

File: description/wheelchair_chassis.xacro (robot description, xacro)
@@ -32,5 +32,5 @@
         <!-- FOR EVERY VISUAL, INCLUDE THE FOLLOWING TO REFLECT IT ON GAZEBO -->
         <gazebo reference="${name}">
-            <material value="Gazebo/White"/>
+            <material value="Gazebo/Grey"/>
         </gazebo>
   <!-- Chassis -->

File: description/wheelchair_footrest.xacro (robot description, xacro)
@@ -34,5 +34,5 @@
         <!-- FOR EVERY VISUAL, INCLUDE THE FOLLOWING TO REFLECT IT ON GAZEBO -->
         <gazebo reference="${side}_footrest">
-            <material value="Gazebo/White"/>
+            <material value="Gazebo/DarkGrey"/>
         </gazebo>
     </xacro:macro>

File: description/wheelchair_lidar.xacro (robot description, xacro)
@@ -62,7 +62,7 @@
             <material>Gazebo/Red</material>
             <!-- type ray is a gazebo type -->
-            <sensor name="laser" type="ray">
+            <!-- <sensor name="laser" type="ray"> -->
                 <!-- place it at the origin of the reference -->
-                <pose> 0 0 0 0 0 0 </pose>
+                <!-- <pose> 0 0 0 0 0 0 </pose>
                 <visualize>true</visualize>
                 <update_rate>10</update_rate>
@@ -79,16 +79,16 @@
                         <max>12</max>
                     </range>
-                </ray>
+                </ray> -->
                 <!-- plugin to make gazebo speak with ros -->
-                <plugin name="laser_controller" filename="libgazebo_ros_ray_sensor.so">
-                    <ros>
+                <!-- <plugin name="laser_controller" filename="libgazebo_ros_ray_sensor.so">
+                    <ros> -->
                         <!-- topic = "scan" -->
-                        <argument>~/out:=scan</argument>
+                        <!-- <argument>~/out:=scan</argument>
                     </ros>
-                    <output_type>sensor_msgs/LaserScan</output_type>
+                    <output_type>sensor_msgs/LaserScan</output_type> -->
                     <!-- will be put in the message of type <output_type>-->
-                    <frame_name>laser_frame</frame_name>
+                    <!-- <frame_name>laser_frame</frame_name>
                 </plugin>
-            </sensor>
+            </sensor> -->
         </gazebo>
     </xacro:macro>

File: description/wheelchair_seat.xacro (robot description, xacro)
@@ -27,5 +27,5 @@
         <!-- FOR EVERY VISUAL, INCLUDE THE FOLLOWING TO REFLECT IT ON GAZEBO -->
         <gazebo reference="${name}">
-            <material value="Gazebo/White"/>
+            <material value="Gazebo/Grey"/>
         </gazebo>
     </xacro:macro>
